Commit message: add camera to the robot

File: irobot/scout_ros2/scout_simulation/robots/scout_mini/scout_mini.urdf (robot description, URDF)
Before this commit: robot scout_mini, 9 links, 8 joints
Links:
- added link camera_link, mass 1e-5; collision box size=0.05 0.05 0.05; visual mesh filename=package://scout_simulation/robots/scout_mini/meshes/d435.dae
- added link camera_link_optical
Joints:
- added joint camera_joint: type fixed, parent base_link, child camera_link, origin xyz=0.2 0.0 0.1 rpy=0 0 1.570796, axis 0 0 0
- added joint camera_optical_joint: type fixed, parent camera_link, child camera_link_optical, origin xyz=0 0 0 rpy=-1.5707963267948966 0 -1.5707963267948966

Commit message: update object detection for project 2

File: irobot/scout_ros2/scout_simulation/robots/scout_mini/scout_mini.urdf (robot description, URDF)
Before this commit: robot scout_mini, 11 links, 10 joints
Links:
- removed link camera_link
- removed link camera_link_optical
- added link camera_left_link, mass 1e-5; collision box size=0.05 0.05 0.05; visual mesh filename=package://bunker_simulation/robots/bunker/meshes/d435.dae
- added link camera_left_link_optical
Joints:
- removed joint camera_joint
- removed joint camera_optical_joint
- added joint camera_left_joint: type fixed, parent base_link, child camera_left_link, origin xyz=0.2 0.0 0.1 rpy=0 0 0, axis 0 0 0
- added joint camera_optical_left_joint: type fixed, parent camera_left_link, child camera_left_link_optical, origin xyz=0 0 0 rpy=-1.5707963267948966 0 -1.5707963267948966

Commit message: update velodyne

File: irobot/scout_ros2/scout_simulation/robots/scout_mini/scout_mini.urdf (robot description, URDF)
Before this commit: robot scout_mini, 11 links, 10 joints
Links:
- removed link camera_left_link
- removed link camera_left_link_optical
Joints:
- removed joint camera_left_joint
- removed joint camera_optical_left_joint

Commit message: add camera and new world

File: irobot/scout_ros2/scout_simulation/robots/scout_mini/scout_mini.urdf (robot description, URDF)
Before this commit: robot scout_mini, 9 links, 8 joints
Links:
- added link camera_link, mass 1e-5; collision box size=0.05 0.05 0.05; visual mesh filename=package://scout_simulation/robots/scout_mini/meshes/d435.dae
- added link camera_link_optical
Joints:
- added joint camera_joint: type fixed, parent base_link, child camera_link, origin xyz=0.2 0.0 0.15 rpy=0 0 0, axis 0 0 0
- added joint camera_optical_joint: type fixed, parent camera_link, child camera_link_optical, origin xyz=0 0 0 rpy=-1.5707963267948966 0 -1.5707963267948966
