Commit message: update

File: irobot/zed/zed-ros2-wrapper/zed_wrapper/urdf/zed_descr.urdf.xacro (robot description, xacro)
@@ -18,29 +18,13 @@
   <xacro:arg name="camera_name"   default="zed" />
   <xacro:arg name="camera_model"  default="zed" />
-  <xacro:arg name="base_frame"    default="base_link" />
-  <xacro:arg name="cam_pos_x"     default="0.0" />
-  <xacro:arg name="cam_pos_y"     default="0.0" />
-  <xacro:arg name="cam_pos_z"     default="0.0" />
-  <xacro:arg name="cam_roll"      default="0.0" />
-  <xacro:arg name="cam_pitch"     default="0.0" />
-  <xacro:arg name="cam_yaw"       default="0.0" />
-  <xacro:arg name="gnss_frame"    default="" />
+  <xacro:arg name="custom_baseline"  default="0.0" />
+  <!-- If GNSS fusion is enabled the position of the antenna with respect to the camera mount point is required -->
+  <xacro:arg name="enable_gnss"   default="false" />
+  <xacro:arg name="gnss_x" default="0.0" />
+  <xacro:arg name="gnss_y" default="0.0" />
+  <xacro:arg name="gnss_z" default="0.0" />
   <xacro:include filename="$(find zed_wrapper)/urdf/zed_macro.urdf.xacro" />
-  <xacro:zed_camera name="$(arg camera_name)" model="$(arg camera_model)" parent="$(arg base_frame)">
-    <origin
-      xyz="$(arg cam_pos_x) $(arg cam_pos_y) $(arg cam_pos_z)"
-      rpy="$(arg cam_roll) $(arg cam_pitch) $(arg cam_yaw)"
-    />
+  <xacro:zed_camera name="$(arg camera_name)" model="$(arg camera_model)" custom_baseline="$(arg custom_baseline)" enable_gnss="$(arg enable_gnss)">
+	    <origin xyz="$(arg gnss_x) $(arg gnss_y) $(arg gnss_z)" rpy="0 0 0"/>
   </xacro:zed_camera>
-  <link name="$(arg base_frame)" />
-  <xacro:property name="gnss_frame" value="$(arg gnss_frame)"/>
-  <!-- Set the position of the GNSS sensor relative to base_link if used -->
-  <xacro:if value="${gnss_frame != ''}">
-    <link name="$(arg gnss_frame)" />
-    <joint name="$(arg gnss_frame)_joint" type="fixed">
-      <parent link="$(arg base_frame)"/>
-      <child link="$(arg gnss_frame)"/>
-      <origin xyz="0 0 0.5" rpy="0 0 0" />
-    </joint>
-  </xacro:if>
 </robot>

File: irobot/zed/zed-ros2-wrapper/zed_wrapper/urdf/zed_macro.urdf.xacro (robot description, xacro)
@@ -21,9 +21,8 @@
     Parameters:
       - name: the camera's name.  should match the parameter sent to the launch file for this camera
-      - model: the tye of camera, one of zed, zedm, zed2, zed2i
-      - parent: the parent link of the camera.  must be defined in the URDF file that uses this macro
-      - origin: the xyz/rpy offset from the parent link
+      - model: the type of camera, one of zed, zedm, zed2, zed2i, zedx, zedxm, virtual
+      - enable_gnss: if true enable the URDF link
   -->
-  <xacro:macro name="zed_camera" params="name=zed model=zed parent *origin">
+  <xacro:macro name="zed_camera" params="name=zed model=zed enable_gnss=false custom_baseline=0 *gnss_origin">
     <xacro:if value="${model == 'zed'}">
       <xacro:property name="baseline" value="0.12" />
@@ -74,33 +73,55 @@
       <xacro:property name="optical_offset_x" value="-0.01" />
     </xacro:if>
+    <xacro:if value="${model == 'virtual'}">
+      <xacro:property name="baseline" value="${custom_baseline}" />
+      <xacro:property name="height" value="0.031" />
+      <xacro:property name="bottom_slope" value="0.0" />
+      <xacro:property name="screw_offset_x" value="0.00" />
+      <xacro:property name="screw_offset_z" value="-0.0155" />
+      <xacro:property name="optical_offset_x" value="0.0" />
+    </xacro:if>
     <!-- Camera mounting point (the threaded screw hole in the bottom) -->
-    <link name="${name}_base_link" />
-    <joint name="${name}_base_joint" type="fixed">
-      <parent link="${parent}"/>
-      <child link="${name}_base_link"/>
-      <xacro:insert_block name="origin" />
-    </joint>
+    <link name="${name}_camera_link" />
     <!-- Camera Center -->
     <link name="${name}_camera_center">
-      <visual>
-        <origin xyz="${screw_offset_x} 0 ${screw_offset_z}" rpy="0 0 0"/>
-        <geometry>
-          <mesh filename="package://zed_interfaces/meshes/${model}.stl" />
-        </geometry>
-        <material name="${model}_mat" />
-      </visual>
-      <collision>
-        <geometry>
-          <mesh filename="package://zed_interfaces/meshes/${model}.stl" />
-        </geometry>
-      </collision>
+      <xacro:unless value="${model == 'virtual'}">
+        <visual>
+          <origin xyz="${screw_offset_x} 0 ${screw_offset_z}" rpy="0 0 0"/>
+          <geometry>
+            <mesh filename="package://zed_interfaces/meshes/${model}.stl" />
+          </geometry>
+          <material name="${model}_mat" />
+        </visual>
+        <collision>
+          <origin xyz="${screw_offset_x} 0 ${screw_offset_z}" rpy="0 0 0"/>
+          <geometry>
+            <mesh filename="package://zed_interfaces/meshes/${model}.stl" />
+          </geometry>
+        </collision>
+      </xacro:unless>
     </link>
     <joint name="${name}_camera_center_joint" type="fixed">
-      <parent link="${name}_base_link"/>
+      <parent link="${name}_camera_link"/>
       <child link="${name}_camera_center"/>
       <origin xyz="0 0 ${height/2}" rpy="0 ${bottom_slope} 0" />
     </joint>
     <!-- Left Camera -->
-    <link name="${name}_left_camera_frame" />
+    <link name="${name}_left_camera_frame">
+      <xacro:if value="${model == 'virtual'}">
+        <visual>
+          <origin xyz="0 0 0" rpy="0 0 0"/>
+          <geometry>
+            <mesh filename="package://zed_interfaces/meshes/${model}.stl" />
+          </geometry>
+          <material name="${model}_mat" />
+        </visual>
+        <collision>
+          <origin xyz="0 0 0" rpy="0 0 0"/>
+          <geometry>
+            <mesh filename="package://zed_interfaces/meshes/${model}.stl" />
+          </geometry>
+        </collision>
+      </xacro:if>
+    </link>
     <joint name="${name}_left_camera_joint" type="fixed">
       <parent link="${name}_camera_center"/>
@@ -115,5 +136,21 @@
     </joint>
     <!-- Right Camera -->
-    <link name="${name}_right_camera_frame" />
+    <link name="${name}_right_camera_frame">
+      <xacro:if value="${model == 'virtual'}">
+        <visual>
+          <origin xyz="0 0 0" rpy="0 0 0"/>
+          <geometry>
+            <mesh filename="package://zed_interfaces/meshes/${model}.stl" />
+          </geometry>
+          <material name="${model}_mat" />
+        </visual>
+        <collision>
+          <origin xyz="0 0 0" rpy="0 0 0"/>
+          <geometry>
+            <mesh filename="package://zed_interfaces/meshes/${model}.stl" />
+          </geometry>
+        </collision>
+      </xacro:if>
+    </link>
     <joint name="${name}_right_camera_joint" type="fixed">
       <parent link="${name}_camera_center"/>
@@ -154,4 +191,12 @@
       </joint>
     </xacro:if>
+    <xacro:if value="${enable_gnss}">
+      <link name="${name}_gnss_link" />
+      <joint name="${name}_gnss_joint" type="fixed">
+        <parent link="${name}_camera_link"/>
+        <child link="${name}_gnss_link"/>
+        <xacro:insert_block name="gnss_origin" />
+      </joint>
+    </xacro:if>
   </xacro:macro>
 </robot>
